File: horizontal-both-sides/horizontal-both-sides.kicad_pcb (KiCad board)
At the start: 2 copper layers, 10.2 x 17.8 mm, 5 parts, among them J1 Grove-I2C-connector, J2 Conn_01x04, J3 Conn_01x04

Commit message: Update each projects for kicad6
Other:
- net class Default removed
