File: horizontal-one-line/horizontal-one-line.kicad_pcb (KiCad board)
At the start: 2 copper layers, 11 x 12.6 mm, 4 parts, among them J1 Grove-I2C-connector, J2 Conn_01x04

Commit message: Update each projects for kicad6
Other:
- net class Default removed
