File: vertical-both-sides/vertical-both-sides.sch (KiCad schematic (older format))
At the start: 3 parts, among them J1 Grove-I2C-connector, J2 Conn_01x02, J3 Conn_01x02

Commit message: Update silk lines for rev2021.02
Parts:
- J1: footprint Connector:NS-Tech_Grove_1x04_P2mm_Vertical -> my-kicad-footprints:NS-Tech_Grove_1x04_P2mm_Vertical_silk_inside
- J2: footprint Connector_PinHeader_2.54mm:PinHeader_1x02_P2.54mm_Vertical -> my-kicad-footprints:PinHeader_1x02_P2.54mm_Vertical_silk_inside
- J3: footprint Connector_PinHeader_2.54mm:PinHeader_1x02_P2.54mm_Vertical -> my-kicad-footprints:PinHeader_1x02_P2.54mm_Vertical_all_circle_silk_inside
Changed lines of the file:
@@
 F 0 "J1" H 3782 3967 50  0000 C CNN
 F 1 "Grove-I2C-connector" H 3782 3876 50  0000 C CNN
-F 2 "Connector:NS-Tech_Grove_1x04_P2mm_Vertical" H 3700 3550 50  0001 C CNN
+F 2 "my-kicad-footprints:NS-Tech_Grove_1x04_P2mm_Vertical_silk_inside" H 3700 3550 50  0001 C CNN
 F 3 "" H 3700 3550 50  0001 C CNN
 	1    3700 3550
@@
 F 0 "J2" H 4230 3392 50  0000 L CNN
 F 1 "Conn_01x02" H 4230 3301 50  0000 L CNN
-F 2 "Connector_PinHeader_2.54mm:PinHeader_1x02_P2.54mm_Vertical" H 4150 3400 50  0001 C CNN
+F 2 "my-kicad-footprints:PinHeader_1x02_P2.54mm_Vertical_silk_inside" H 4150 3400 50  0001 C CNN
 F 3 "~" H 4150 3400 50  0001 C CNN
 	1    4150 3400
@@
 F 0 "J3" H 4230 3592 50  0000 L CNN
 F 1 "Conn_01x02" H 4230 3501 50  0000 L CNN
-F 2 "Connector_PinHeader_2.54mm:PinHeader_1x02_P2.54mm_Vertical" H 4150 3600 50  0001 C CNN
+F 2 "my-kicad-footprints:PinHeader_1x02_P2.54mm_Vertical_all_circle_silk_inside" H 4150 3600 50  0001 C CNN
 F 3 "~" H 4150 3600 50  0001 C CNN
 	1    4150 3600
