File: vertical-both-sides/vertical-both-sides.kicad_pcb (KiCad board)
At the start: 2 copper layers, 5.1 x 17.4 mm, 5 parts, among them J1 Grove-I2C-connector, J2 Conn_01x02, J3 Conn_01x02

Commit message: Update each projects for kicad6
Other:
- net class Default removed
