File: vertical-one-line/vertical-one-line.kicad_pcb (KiCad board)
At the start: 2 copper layers, 8.1 x 10.2 mm, 4 parts, among them J1 Grove-I2C-connector, J2 Conn_01x04

Commit message: Update each projects for kicad6
Other:
- net class Default removed
